Commit message: Add correct urdf (previous was wrong)

File: osgMinitaur/quadruped2Odie.urdf (robot description, URDF)
Before this commit: robot quadruped, 25 links, 24 joints
Links:
- added link foot_back_left_link, mass 0.001; collision sphere radius=0.0125; visual sphere radius=0.0125
- added link foot_back_right_link, mass 0.001; collision sphere radius=0.0125; visual sphere radius=0.0125
- added link foot_front_left_link, mass 0.001; collision sphere radius=0.0125; visual sphere radius=0.0125
- added link foot_front_right_link, mass 0.001; collision sphere radius=0.0125; visual sphere radius=0.0125
- added link rotor_tail, mass 0.398; collision cylinder length=0.026 radius=0.0434; visual cylinder length=0.026 radius=0.0434
- added link stator_back_leftL_link, mass 0.398; collision box size=0.06 0.06 0.02; visual box size=0.06 0.06 0.02
- added link stator_back_leftR_link, mass 0.398; collision box size=0.06 0.06 0.02; visual box size=0.06 0.06 0.02
- added link stator_back_rightL_link, mass 0.398; collision box size=0.06 0.06 0.02; visual box size=0.06 0.06 0.02
- added link stator_back_rightR_link, mass 0.398; collision box size=0.06 0.06 0.02; visual box size=0.06 0.06 0.02
- added link stator_front_leftL_link, mass 0.398; collision box size=0.06 0.06 0.02; visual box size=0.06 0.06 0.02
- added link stator_front_leftR_link, mass 0.398; collision box size=0.06 0.06 0.02; visual box size=0.06 0.06 0.02
- added link stator_front_rightL_link, mass 0.398; collision box size=0.06 0.06 0.02; visual box size=0.06 0.06 0.02
- added link stator_front_rightR_link, mass 0.398; collision box size=0.06 0.06 0.02; visual box size=0.06 0.06 0.02
- added link stator_tail, mass 0.398; collision box size=0.06 0.06 0.02; visual box size=0.06 0.06 0.02
- link lower_leg_back_leftL_link: mass 0.05186 -> 0.043; geometry collision box size=.01 0.01 .2275; visual box size=.01 0.01 .2275
- link lower_leg_back_leftR_link: mass 0.043 -> 0.05186
- link lower_leg_back_rightR_link: geometry collision box size=.01 0.01 0.2275; visual box size=.01 0.01 0.2275
- link lower_leg_front_leftL_link: mass 0.05186 -> 0.043; geometry collision box size=.01 0.01 .2275; visual box size=.01 0.01 .2275
- link lower_leg_front_leftR_link: mass 0.043 -> 0.05186
- link lower_leg_front_rightR_link: geometry collision box size=.01 0.01 .2275; visual box size=.01 0.01 .2275
- link motor_back_leftL_link: mass 0.398 -> 0.00001
- link motor_back_leftR_link: mass 0.398 -> 0.00001
- link motor_back_rightL_link: mass 0.398 -> 0.00001
- link motor_back_rightR_link: mass 0.398 -> 0.00001
- link motor_front_leftL_link: mass 0.398 -> 0.00001
- link motor_front_leftR_link: mass 0.398 -> 0.00001
- link motor_front_rightL_link: mass 0.398 -> 0.00001
- link motor_front_rightR_link: mass 0.398 -> 0.00001
Joints:
- removed joint hip_front_leftR_link
- removed joint hip_leftR_link
- removed joint motor_back_leftL_link
- removed joint motor_front_leftL_link
- added joint hip_front_leftL_link: type fixed, parent motor_front_leftL_link, child upper_leg_front_leftL_link, origin xyz=0.0 0.06 0.02 rpy=-1.57075 0 0, axis 0 0 1, limit effort=100 velocity=1000
- added joint hip_leftL_link: type fixed, parent motor_back_leftL_link, child upper_leg_back_leftL_link, origin xyz=0.0 0.06 0.02 rpy=-1.57075 0 0, axis 0 0 1, limit effort=100 velocity=1000
- added joint motor_back_leftR_link: type fixed, parent motor_back_leftR_link, child upper_leg_back_leftR_link, origin xyz=0.0 0.06 -0.02 rpy=-1.57075 0 0, axis 0 0 1, limit effort=100 velocity=1000
- added joint motor_front_leftR_link: type fixed, parent motor_front_leftR_link, child upper_leg_front_leftR_link, origin xyz=0.0 0.06 -0.02 rpy=-1.57075 0 0, axis 0 0 1, limit effort=100 velocity=1000
- added joint rotor_tail_joint: type continuous, parent stator_tail, child rotor_tail, origin xyz=0.0 0 -0.025 rpy=0 0 3.14159, axis 0 0 1, limit effort=100 velocity=1000
- added joint stator_back_leftL_joint: type fixed, parent base_chassis_link, child stator_back_leftL_link, origin xyz=-0.21 0.165 0 rpy=1.57075 0 0, axis 0 0 1, limit effort=100 velocity=1000
- added joint stator_back_leftR_joint: type fixed, parent base_chassis_link, child stator_back_leftR_link, origin xyz=-0.21 0.055 0 rpy=1.57075 0 0, axis 0 0 1, limit effort=100 velocity=1000
- added joint stator_back_rightL_joint: type fixed, parent base_chassis_link, child stator_back_rightL_link, origin xyz=-0.21 -0.055 0 rpy=1.57075 0 0, axis 0 0 1, limit effort=100 velocity=1000
- added joint stator_back_rightR_joint: type fixed, parent base_chassis_link, child stator_back_rightR_link, origin xyz=-0.21 -0.165 0 rpy=1.57075 0 0, axis 0 0 1, limit effort=100 velocity=1000
- added joint stator_front_leftL_joint: type fixed, parent base_chassis_link, child stator_front_leftL_link, origin xyz=0.21 0.165 0 rpy=1.57075 0 0, axis 0 0 1, limit effort=100 velocity=1000
- added joint stator_front_leftR_joint: type fixed, parent base_chassis_link, child stator_front_leftR_link, origin xyz=0.21 0.055 0 rpy=1.57075 0 0, axis 0 0 1, limit effort=100 velocity=1000
- added joint stator_front_rightL_joint: type fixed, parent base_chassis_link, child stator_front_rightL_link, origin xyz=0.21 -0.055 0 rpy=1.57075 0 0, axis 0 0 1, limit effort=100 velocity=1000
- added joint stator_front_rightR_joint: type fixed, parent base_chassis_link, child stator_front_rightR_link, origin xyz=0.21 -0.165 0 rpy=1.57075 0 0, axis 0 0 1, limit effort=100 velocity=1000
- added joint stator_tail_joint: type fixed, parent base_chassis_link, child stator_tail, origin xyz=0.0 -0.05 0.1 rpy=1.57075 0 0, axis 0 0 1, limit effort=100 velocity=1000
- added joint toe_back_left_link: type fixed, parent lower_leg_back_leftL_link, child foot_back_left_link, origin xyz=0.0 0.0 0.2275 rpy=0 0 0, axis 0 1 0, limit effort=100 velocity=1000
- added joint toe_back_right_link: type fixed, parent lower_leg_back_rightR_link, child foot_back_right_link, origin xyz=0.0 0.0 0.2275 rpy=0 0 0, axis 0 1 0, limit effort=100 velocity=1000
- added joint toe_front_left_link: type fixed, parent lower_leg_front_leftL_link, child foot_front_left_link, origin xyz=0.0 0.0 0.2275 rpy=0 0 0, axis 0 1 0, limit effort=100 velocity=1000
- added joint toe_front_right_link: type fixed, parent lower_leg_front_rightR_link, child foot_front_right_link, origin xyz=0.0 0.0 0.2275 rpy=0 0 0, axis 0 1 0, limit effort=100 velocity=1000
- joint motor_back_leftL_joint: origin xyz=-0.21 0.06 0 rpy=1.57075 0 0 -> xyz=-0.21 0.14 0 rpy=1.57075 0 0
- joint motor_back_leftR_joint: origin xyz=-0.21 0.125 0 rpy=1.57075 0 0 -> xyz=-0.21 0.08 0 rpy=-1.57075 0 0
- joint motor_back_rightL_joint: origin xyz=-0.21 -0.06 0 rpy=1.57075 0 0 -> xyz=-0.21 -0.08 0 rpy=-1.57075 0 0
- joint motor_back_rightR_joint: origin xyz=-0.21 -0.125 0 rpy=1.57075 0 0 -> xyz=-0.21 -0.14 0 rpy=1.57075 0 0
- joint motor_front_leftL_joint: origin xyz=0.21 0.06 0 rpy=1.57075 0 0 -> xyz=0.21 0.14 0 rpy=1.57075 0 0
- joint motor_front_leftR_joint: origin xyz=0.21 0.125 0 rpy=1.57075 0 0 -> xyz=0.21 0.08 0 rpy=-1.57075 0 0
- joint motor_front_rightL_joint: origin xyz=0.21 -0.06 0 rpy=1.57075 0 0 -> xyz=0.21 -0.08 0 rpy=-1.57075 0 0
- joint motor_front_rightR_joint: origin xyz=0.21 -0.125 0 rpy=1.57075 0 0 -> xyz=0.21 -0.14 0 rpy=1.57075 0 0
